File: 2.Charger-Buck Boost/2.Charger-Buck Boost.sch (KiCad schematic (older format))
At the start: 1 part

Commit message: Added Charging circuit with footprint, Power input Note
Parts:
- removed BD?: BlockDiagram, symbol KiCAD~Demo:BlockDiagram
Changed lines of the file:
@@
 $Descr A4 11693 8268
 encoding utf-8
-Sheet 1 1
+Sheet 1 2
 Title ""
 Date "2020-07-26"
@@
 Comment4 ""
 $EndDescr
-$Comp
-L KiCAD~Demo:BlockDiagram BD?
-U 1 1 5F1D5706
-P 4900 4750
-F 0 "BD?" H 5300 5100 59  0001 C CNN
-F 1 "BlockDiagram" H 5300 5100 59  0001 C CNN
-F 2 "" H 5300 5100 59  0001 C CNN
-F 3 "" H 5300 5100 59  0001 C CNN
-	1    4900 4750
-	1    0    0    -1
-$EndComp
 Text Notes 4950 4900 0    79   ~ 16
 TPS63802
@@
 Text Notes 6200 4550 0    47   ~ 0
 2.5A
+$Sheet
+S 12000 800  1600 900
+U 5F1E11EF
+F0 "Charger+BuckBoost" 50
+F1 "file5F1E11EE.sch" 50
+$EndSheet
 $EndSCHEMATC
